Commit message: Working Locomotion and Sim

File: src/teleop_robot/urdf/my_robot.urdf.xacro (robot description, xacro)
@@ -4,23 +4,6 @@
     <xacro:include filename="$(find teleop_robot)/urdf/my_robot_links.xacro"/>
     <xacro:include filename="$(find teleop_robot)/urdf/my_robot_joints.xacro"/>
-    <ros2_control name="GZ_DiffDriveRobot" type="system">
-      <hardware>
-        <plugin>gazebo_ros2_control/GazeboSystem</plugin>
-      </hardware>
-      <joint name="right_wheel_joint">
-          <command_interface name="velocity"/>
-          <state_interface name="velocity"/>
-          <state_interface name="position"/>
-      </joint>
-      <joint name="left_wheel_joint">
-          <command_interface name="velocity"/>
-          <state_interface name="velocity"/>
-          <state_interface name="position"/>
-      </joint>
-    </ros2_control>
-    <gazebo>
-        <plugin name="gazebo_ros2_control" filename="libgazebo_ros2_control.so">
-            <!-- <parameters>$(find teleop_robot)/config/my_controllers.yaml</parameters> -->
-        </plugin>
-    </gazebo>
+    <xacro:include filename="$(find teleop_robot)/urdf/ros2_control.xacro"/>
+    <xacro:include filename="$(find teleop_robot)/urdf/lidar.xacro"/>
+    <xacro:lidar parent_link="base_link" x_loc="0.0" y_loc="0.0" z_loc="0.15"/>
 </robot>

File: src/teleop_robot/urdf/robot_properties.xacro (robot description, xacro)
@@ -8,4 +8,6 @@
     <xacro:property name="chassis_mass" value="2.0" />
     <xacro:property name="wheel_mass" value="0.5" />
+    <xacro:property name="M_PI" value="3.14159265359"/>
+    <xacro:property name="DEG_TO_RAD" value="${M_PI / 180.0}"/>
     <material name="blue">
         <color rgba="0 0 0.8 1"/>
@@ -13,4 +15,7 @@
     <material name="grey">
         <color rgba="0.5 0.5 0.5 1"/>
+    </material>
+    <material name="black">
+        <color rgba="0 0 0 0"/>
     </material>
     <xacro:macro name="box_inertia" params="m l w h">
