Commit message: Remove build artifacts from tracking and update .gitignore
- Remove src/build/, src/install/, src/log/ from git tracking
- Update .gitignore to cover root and src-level build artifacts, .DS_Store, and Claude Code files
- Add Ignition Gazebo support (sim_ign launch, ign xacro variants, warehouse world)
- Tune wheel joint limits (effort 100, velocity 20) and add damping/friction
- Install worlds directory in CMakeLists.txt
- Add requirements.txt

File: src/teleop_robot/urdf/my_robot_joints.xacro (robot description, xacro)
@@ -6,5 +6,6 @@
         <origin xyz="${0.25 - wheel_radius*2} ${-0.25- wheel_length/2} -0.10" rpy="${pi/2} 0 0"/>
         <axis xyz="0 0 -1"/>
-        <limit effort="10" velocity="0.1"/>
+        <limit effort="100" velocity="20"/>
+        <dynamics damping="0.1" friction="0.1"/>
     </joint>
     <joint name="left_wheel_joint" type="continuous">
@@ -13,5 +14,6 @@
         <origin xyz="${0.25 - wheel_radius*2} ${0.25+ wheel_length/2} -0.10" rpy="${pi/2} 0 0"/>
         <axis xyz="0 0 -1"/>
-        <limit effort="10" velocity="0.1"/>
+        <limit effort="100" velocity="20"/>
+        <dynamics damping="0.1" friction="0.1"/>
     </joint>
     <joint name="castor_joint" type="fixed">
